Commit message: update for macro template

File: summit_xl_description/urdf/arms/franka/fr3.urdf.xacro (robot description, xacro)
@@ -1,8 +1,10 @@
 <?xml version='1.0' encoding='utf-8'?>
 <robot xmlns:xacro="http://www.ros.org/wiki/xacro" name="fr3">
+  <xacro:macro name="franka_pre" params = "prefix">
   <xacro:include filename="$(find summit_xl_description)/urdf/arms/franka/franka_robot.xacro"/>
-  <xacro:arg name="arm_id" default="fr3" />
-  <xacro:franka_robot arm_id="$(arg arm_id)"
+  <xacro:arg name="arm_id" default="fr3"/>
+  <xacro:franka_robot prefix = "${prefix}" arm_id="${prefix}_fr3"
                       joint_limits="${xacro.load_yaml('$(find summit_xl_description)/urdf/arms/franka/joint_limits.yaml')}">
   </xacro:franka_robot>
+  </xacro:macro>
 </robot>

File: summit_xl_description/urdf/arms/franka/franka_robot.xacro (robot description, xacro)
@@ -1,5 +1,5 @@
 <?xml version='1.0' encoding='utf-8'?>
 <robot xmlns:xacro="http://www.ros.org/wiki/xacro">
-  <xacro:macro name="franka_robot" params="arm_id joint_limits">
+  <xacro:macro name="franka_robot" params="prefix arm_id joint_limits">
     <!-- Name of this panda -->
     <!-- Should a franka_gripper be mounted at the flange?" -->
@@ -17,9 +17,9 @@
       <xacro:include filename="$(find summit_xl_description)/urdf/arms/franka/franka_hand.xacro"/>
       <xacro:franka_hand
-          arm_id="$(arg arm_id)"
+          arm_id="${prefix}_$(arg arm_id)"
           rpy="0 0 ${-pi/4}"
           tcp_xyz="$(arg tcp_xyz)"
           tcp_rpy="$(arg tcp_rpy)"
-          connected_to="$(arg arm_id)_link8"
+          connected_to="${prefix}_$(arg arm_id)_link8"
           safety_distance="0.03"
           gazebo="$(arg gazebo)"

File: summit_xl_description/urdf/structures/d435.urdf.xacro (robot description, xacro)
@@ -1,9 +1,9 @@
 <?xml version="1.0"?>
 <robot xmlns:xacro="http://ros.org/wiki/xacro" name="sensor_d435">
-  <xacro:macro name="sensor_d435" params="*origin parent name:=camera use_nominal_extrinsics:=false">
+  <xacro:macro name="sensor_d435" params="*origin prefix parent name:=camera use_nominal_extrinsics:=false">
     <xacro:property name="M_PI" value="3.1415926535897931"/>
-    <material name="aluminum">
+    <!-- <material name="aluminum">
       <color rgba="0.5 0.5 0.5 1"/>
-    </material>
+    </material> -->
     <!-- The following values are approximate, and the camera node
      publishing TF values with actual calibrated camera extrinsic values -->
@@ -30,16 +30,16 @@
     <xacro:property name="d435_cam_depth_pz" value="${d435_cam_height/2}"/>
     <!-- camera body, with origin at bottom screw mount -->
-    <joint name="${name}_joint" type="fixed">
+    <joint name="${prefix}_${name}_joint" type="fixed">
       <xacro:insert_block name="origin" />
       <parent link="${parent}"/>
-      <child link="${name}_bottom_screw_frame" />
+      <child link="${prefix}_${name}_bottom_screw_frame" />
     </joint>
-    <link name="${name}_bottom_screw_frame"/>
-    <joint name="${name}_link_joint" type="fixed">
+    <link name="${prefix}_${name}_bottom_screw_frame"/>
+    <joint name="${prefix}_${name}_link_joint" type="fixed">
       <origin xyz="${d435_mesh_x_offset} ${d435_cam_depth_py} ${d435_cam_depth_pz}" rpy="0 0 0"/>
-      <parent link="${name}_bottom_screw_frame"/>
-      <child link="${name}_link" />
+      <parent link="${prefix}_${name}_bottom_screw_frame"/>
+      <child link="${prefix}_${name}_link" />
     </joint>
-    <link name="${name}_link">
+    <link name="${prefix}_${name}_link">
       <visual>
         <origin xyz="${d435_zero_depth_to_glass + d435_glass_to_front} ${-d435_cam_depth_py} 0" rpy="${M_PI/2} 0 ${M_PI/2}"/>
@@ -63,60 +63,60 @@
     <!--xacro:if value="$(arg use_nominal_extrinsics)"-->
     <!-- camera depth joints and links -->
-    <joint name="${name}_depth_joint" type="fixed">
+    <joint name="${prefix}_${name}_depth_joint" type="fixed">
       <origin xyz="0 0 0" rpy="0 0 0"/>
-      <parent link="${name}_link"/>
-      <child link="${name}_depth_frame" />
+      <parent link="${prefix}_${name}_link"/>
+      <child link="${prefix}_${name}_depth_frame" />
     </joint>
-    <link name="${name}_depth_frame"/>
-    <joint name="${name}_depth_optical_joint" type="fixed">
+    <link name="${prefix}_${name}_depth_frame"/>
+    <joint name="${prefix}_${name}_depth_optical_joint" type="fixed">
       <origin xyz="0 0 0" rpy="${-M_PI/2} 0 ${-M_PI/2}" />
-      <parent link="${name}_depth_frame" />
-      <child link="${name}_depth_optical_frame" />
+      <parent link="${prefix}_${name}_depth_frame" />
+      <child link="${prefix}_${name}_depth_optical_frame" />
     </joint>
-    <link name="${name}_depth_optical_frame"/>
+    <link name="${prefix}_${name}_depth_optical_frame"/>
     <!-- camera left IR joints and links -->
-    <joint name="${name}_infra1_joint" type="fixed">
+    <joint name="${prefix}_${name}_infra1_joint" type="fixed">
       <origin xyz="0 ${d435_cam_depth_to_infra1_offset} 0" rpy="0 0 0" />
-      <parent link="${name}_link" />
-      <child link="${name}_infra1_frame" />
+      <parent link="${prefix}_${name}_link" />
+      <child link="${prefix}_${name}_infra1_frame" />
     </joint>
-    <link name="${name}_infra1_frame"/>
-    <joint name="${name}_infra1_optical_joint" type="fixed">
+    <link name="${prefix}_${name}_infra1_frame"/>
+    <joint name="${prefix}_${name}_infra1_optical_joint" type="fixed">
       <origin xyz="0 0 0" rpy="${-M_PI/2} 0 ${-M_PI/2}" />
-      <parent link="${name}_infra1_frame" />
-      <child link="${name}_infra1_optical_frame" />
+      <parent link="${prefix}_${name}_infra1_frame" />
+      <child link="${prefix}_${name}_infra1_optical_frame" />
     </joint>
-    <link name="${name}_infra1_optical_frame"/>
+    <link name="${prefix}_${name}_infra1_optical_frame"/>
     <!-- camera right IR joints and links -->
-    <joint name="${name}_infra2_joint" type="fixed">
+    <joint name="${prefix}_${name}_infra2_joint" type="fixed">
       <origin xyz="0 ${d435_cam_depth_to_infra2_offset} 0" rpy="0 0 0" />
-      <parent link="${name}_link" />
-      <child link="${name}_infra2_frame" />
+      <parent link="${prefix}_${name}_link" />
+      <child link="${prefix}_${name}_infra2_frame" />
     </joint>
-    <link name="${name}_infra2_frame"/>
-    <joint name="${name}_infra2_optical_joint" type="fixed">
+    <link name="${prefix}_${name}_infra2_frame"/>
+    <joint name="${prefix}_${name}_infra2_optical_joint" type="fixed">
       <origin xyz="0 0 0" rpy="${-M_PI/2} 0 ${-M_PI/2}" />
-      <parent link="${name}_infra2_frame" />
-      <child link="${name}_infra2_optical_frame" />
+      <parent link="${prefix}_${name}_infra2_frame" />
+      <child link="${prefix}_${name}_infra2_optical_frame" />
     </joint>
-    <link name="${name}_infra2_optical_frame"/>
+    <link name="${prefix}_${name}_infra2_optical_frame"/>
     <!-- camera color joints and links -->
-    <joint name="${name}_color_joint" type="fixed">
+    <joint name="${prefix}_${name}_color_joint" type="fixed">
       <origin xyz="0 ${d435_cam_depth_to_color_offset} 0" rpy="0 0 0" />
-      <parent link="${name}_link" />
-      <child link="${name}_color_frame" />
+      <parent link="${prefix}_${name}_link" />
+      <child link="${prefix}_${name}_color_frame" />
     </joint>
-    <link name="${name}_color_frame"/>
-    <joint name="${name}_color_optical_joint" type="fixed">
+    <link name="${prefix}_${name}_color_frame"/>
+    <joint name="${prefix}_${name}_color_optical_joint" type="fixed">
       <origin xyz="0 0 0" rpy="${-M_PI/2} 0 ${-M_PI/2}" />
-      <parent link="${name}_color_frame" />
-      <child link="${name}_color_optical_frame" />
+      <parent link="${prefix}_${name}_color_frame" />
+      <child link="${prefix}_${name}_color_optical_frame" />
     </joint>
-    <link name="${name}_color_optical_frame"/>
+    <link name="${prefix}_${name}_color_optical_frame"/>
     <!--/xacro:if-->
     <!-- Gazebo part -->
     <!-- D435 Gazebo -->
-   <gazebo reference="camera_link">
-    <sensor name="camera" type="depth">
+   <gazebo reference="${prefix}_camera_link">
+    <sensor name="${prefix}_camera" type="depth">
       <update_rate>30</update_rate>
       <visualize>true</visualize>

File: summit_xl_description/urdf/structures/roas.urdf.xacro (robot description, xacro)
@@ -1,70 +1,72 @@
 <?xml version="1.0"?>
 <robot xmlns:xacro="http://ros.org/wiki/xacro" name="roas">
-  <xacro:property name="PI" value="3.1415926535897931"/>
-  <xacro:include filename="$(find summit_xl_description)/urdf/structures/d435.urdf.xacro"/>
-  <link name="top_structure">
-    <visual>
-      <origin xyz="0 0 0" rpy="0 0 0" />
-      <geometry>
-        <mesh filename="package://summit_xl_description/meshes/structures/top_structure_roas.STL"/>
-      </geometry>
-      <material name="silver">
-        <color rgba="0.75 0.75 0.75 1"/>
-      </material>
-    </visual>
-    <collision>
+  <xacro:macro name="roas" params="prefix">
+    <xacro:property name="PI" value="3.1415926535897931"/>
+    <xacro:include filename="$(find summit_xl_description)/urdf/structures/d435.urdf.xacro"/>
+    <link name="${prefix}_top_structure">
+      <visual>
+        <origin xyz="0 0 0" rpy="0 0 0" />
+        <geometry>
+          <mesh filename="package://summit_xl_description/meshes/structures/top_structure_roas.STL"/>
+        </geometry>
+        <material name="silver">
+          <color rgba="0.75 0.75 0.75 1"/>
+        </material>
+      </visual>
+      <collision>
+        <origin xyz="0 0 0" rpy="0 0 0"/>
+        <geometry>
+          <mesh filename="package://summit_xl_description/meshes/structures/top_structure_roas.STL"/>
+        </geometry>
+      </collision>
+    </link>
+    <xacro:include filename="$(find summit_xl_description)/urdf/arms/franka/fr3.urdf.xacro"/>
+    <xacro:franka_pre prefix = "${prefix}"/>
+    <joint name="${prefix}_fr3_base_joint" type="fixed">
+      <origin xyz="0.23 0 0.66" rpy="0 0 0"/>
+      <parent link="${prefix}_top_structure"/>
+      <child link="${prefix}_fr3_link0"/>
+    </joint>
+    <link name="${prefix}_ee_link"/>
+    <joint name="${prefix}_ee_joint" type="fixed">
+      <parent link="${prefix}_fr3_link8" />
+      <child link="${prefix}_ee_link" />
       <origin xyz="0 0 0" rpy="0 0 0"/>
-      <geometry>
-        <mesh filename="package://summit_xl_description/meshes/structures/top_structure_roas.STL"/>
-      </geometry>
-    </collision>
-  </link>
-  <xacro:include filename="$(find summit_xl_description)/urdf/arms/franka/fr3.urdf.xacro"/>
-  <!-- fr3 -->
-  <joint name="fr3_base_joint" type="fixed">
-    <origin xyz="0.23 0 0.66" rpy="0 0 0"/>
-    <parent link="top_structure"/>
-    <child link="fr3_link0"/>
-  </joint>
-  <link name="ee_link"/>
-  <joint name="ee_joint" type="fixed">
-    <parent link="fr3_link8" />
-    <child link="ee_link" />
-    <origin xyz="0 0 0" rpy="0 0 0"/>
-  </joint>
-  <!-- D435 -->
-  <xacro:sensor_d435 parent="camera_bracket" name="camera">
-    <origin xyz="0.0377 0 0.0105" rpy="0 -1.57 3.14"/>
-  </xacro:sensor_d435>
-  <link name="d435_link"/>
-  <joint name="d435_joint" type="fixed">
-    <parent link="camera_link"/>
-    <child link="d435_link"/>
-    <origin xyz="0.0 0.0 0.0" rpy="-${PI/2} 0 -${PI/2}"/>
-  </joint>
-  <link name="camera_bracket">
-    <visual>
-      <origin xyz="0 0 0" rpy="0 0 0" />
-      <geometry>
-        <mesh filename="package://summit_xl_description/meshes/structures/hand_camera.STL"/>
-      </geometry>
-      <material name="silver">
-        <color rgba="0.75 0.75 0.75 1"/>
-      </material>
-    </visual>
-    <collision>
-      <origin xyz="0 0 0" rpy="0 0 0" />
-      <geometry>
-        <mesh filename="package://summit_xl_description/meshes/structures/hand_camera.STL"/>
-      </geometry>
-      <material name="silver">
-        <color rgba="0.75 0.75 0.75 1"/>
-      </material>
-    </collision>
-  </link>
-  <joint name="camera_bracket_joint" type="fixed">
-    <parent link="ee_link" />
-    <child link = "camera_bracket" />
-    <origin xyz="0 0 0.003" rpy="0 0 -0.785" />
-  </joint>
+    </joint>
+    <!-- D435 -->
+    <xacro:sensor_d435 parent="${prefix}_camera_bracket" name="camera" prefix ="${prefix}">
+      <origin xyz="0.0377 0 0.0105" rpy="0 -1.57 3.14"/>
+    </xacro:sensor_d435>
+    <link name="${prefix}_d435_link"/>
+    <joint name="${prefix}_d435_joint" type="fixed">
+      <parent link="${prefix}_camera_link"/>
+      <child link="${prefix}_d435_link"/>
+      <origin xyz="0.0 0.0 0.0" rpy="-${PI/2} 0 -${PI/2}"/>
+    </joint>
+    <link name="${prefix}_camera_bracket">
+      <visual>
+        <origin xyz="0 0 0" rpy="0 0 0" />
+        <geometry>
+          <mesh filename="package://summit_xl_description/meshes/structures/hand_camera.STL"/>
+        </geometry>
+        <material name="silver">
+          <color rgba="0.75 0.75 0.75 1"/>
+        </material>
+      </visual>
+      <collision>
+        <origin xyz="0 0 0" rpy="0 0 0" />
+        <geometry>
+          <mesh filename="package://summit_xl_description/meshes/structures/hand_camera.STL"/>
+        </geometry>
+        <material name="silver">
+          <color rgba="0.75 0.75 0.75 1"/>
+        </material>
+      </collision>
+    </link>
+    <joint name="${prefix}_camera_bracket_joint" type="fixed">
+      <parent link="${prefix}_ee_link" />
+      <child link = "${prefix}_camera_bracket" />
+      <origin xyz="0 0 0.003" rpy="0 0 -0.785" />
+    </joint>
+  </xacro:macro>
 </robot>

File: summit_xls/summit_xls_franka_sim/urdf/arm/fr3.urdf.xacro (robot description, xacro)
@@ -1,8 +1,10 @@
 <?xml version='1.0' encoding='utf-8'?>
 <robot xmlns:xacro="http://www.ros.org/wiki/xacro" name="fr3">
-  <xacro:include filename="$(find summit_xls_franka_sim)/urdf/arm/franka_robot.xacro"/>
-  <xacro:arg name="arm_id" default="fr3" />
-  <xacro:franka_robot arm_id="$(arg arm_id)"
-                      joint_limits="${xacro.load_yaml('$(find summit_xls_franka_sim)/urdf/arm/joint_limits.yaml')}">
-  </xacro:franka_robot>
+  <xacro:macro name="fr3" params="prefix">
+    <xacro:include filename="$(find summit_xls_franka_sim)/urdf/arm/franka_robot.xacro"/>
+    <xacro:arg name="arm_id" default="${prefix}_fr3" />
+    <xacro:franka_robot arm_id="$(arg arm_id)"
+                        joint_limits="${xacro.load_yaml('$(find summit_xls_franka_sim)/urdf/arm/joint_limits.yaml')}">
+    </xacro:franka_robot>
+  <xacro:macro>
 </robot>

File: summit_xls/summit_xls_franka_sim/urdf/d435.urdf.xacro (robot description, xacro)
@@ -1,5 +1,5 @@
 <?xml version="1.0"?>
 <robot xmlns:xacro="http://ros.org/wiki/xacro" name="sensor_d435">
-  <xacro:macro name="sensor_d435" params="*origin parent name:=camera use_nominal_extrinsics:=false">
+  <xacro:macro name="sensor_d435" params="*origin prefix parent name:=camera use_nominal_extrinsics:=false">
     <xacro:property name="M_PI" value="3.1415926535897931"/>
     <material name="aluminum">
@@ -30,16 +30,16 @@
     <xacro:property name="d435_cam_depth_pz" value="${d435_cam_height/2}"/>
     <!-- camera body, with origin at bottom screw mount -->
-    <joint name="${name}_joint" type="fixed">
+    <joint name="${prefix}_${name}_joint" type="fixed">
       <xacro:insert_block name="origin" />
       <parent link="${parent}"/>
-      <child link="${name}_bottom_screw_frame" />
+      <child link="${prefix}_${name}_bottom_screw_frame" />
     </joint>
-    <link name="${name}_bottom_screw_frame"/>
+    <link name="${prefix}_${name}_bottom_screw_frame"/>
     <joint name="${name}_link_joint" type="fixed">
       <origin xyz="${d435_mesh_x_offset} ${d435_cam_depth_py} ${d435_cam_depth_pz}" rpy="0 0 0"/>
-      <parent link="${name}_bottom_screw_frame"/>
-      <child link="${name}_link" />
+      <parent link="${prefix}_${name}_bottom_screw_frame"/>
+      <child link="${prefix}_${name}_link" />
     </joint>
-    <link name="${name}_link">
+    <link name="${prefix}_${name}_link">
       <visual>
         <origin xyz="${d435_zero_depth_to_glass + d435_glass_to_front} ${-d435_cam_depth_py} 0" rpy="${M_PI/2} 0 ${M_PI/2}"/>
@@ -63,55 +63,55 @@
     <!--xacro:if value="$(arg use_nominal_extrinsics)"-->
     <!-- camera depth joints and links -->
-    <joint name="${name}_depth_joint" type="fixed">
+    <joint name="${prefix}_${name}_depth_joint" type="fixed">
       <origin xyz="0 0 0" rpy="0 0 0"/>
-      <parent link="${name}_link"/>
-      <child link="${name}_depth_frame" />
+      <parent link="${prefix}_${name}_link"/>
+      <child link="${prefix}_${name}_depth_frame" />
     </joint>
-    <link name="${name}_depth_frame"/>
-    <joint name="${name}_depth_optical_joint" type="fixed">
+    <link name="${prefix}_${name}_depth_frame"/>
+    <joint name="${prefix}_${name}_depth_optical_joint" type="fixed">
       <origin xyz="0 0 0" rpy="${-M_PI/2} 0 ${-M_PI/2}" />
-      <parent link="${name}_depth_frame" />
-      <child link="${name}_depth_optical_frame" />
+      <parent link="${prefix}_${name}_depth_frame" />
+      <child link="${prefix}_${name}_depth_optical_frame" />
     </joint>
-    <link name="${name}_depth_optical_frame"/>
+    <link name="${prefix}_${name}_depth_optical_frame"/>
     <!-- camera left IR joints and links -->
-    <joint name="${name}_infra1_joint" type="fixed">
+    <joint name="${prefix}_${name}_infra1_joint" type="fixed">
       <origin xyz="0 ${d435_cam_depth_to_infra1_offset} 0" rpy="0 0 0" />
-      <parent link="${name}_link" />
-      <child link="${name}_infra1_frame" />
+      <parent link="${prefix}_${name}_link" />
+      <child link="${prefix}_${name}_infra1_frame" />
     </joint>
-    <link name="${name}_infra1_frame"/>
-    <joint name="${name}_infra1_optical_joint" type="fixed">
+    <link name="${prefix}_${name}_infra1_frame"/>
+    <joint name="${prefix}_${name}_infra1_optical_joint" type="fixed">
       <origin xyz="0 0 0" rpy="${-M_PI/2} 0 ${-M_PI/2}" />
-      <parent link="${name}_infra1_frame" />
-      <child link="${name}_infra1_optical_frame" />
+      <parent link="${prefix}_${name}_infra1_frame" />
+      <child link="${prefix}_${name}_infra1_optical_frame" />
     </joint>
-    <link name="${name}_infra1_optical_frame"/>
+    <link name="${prefix}_${name}_infra1_optical_frame"/>
     <!-- camera right IR joints and links -->
-    <joint name="${name}_infra2_joint" type="fixed">
+    <joint name="${prefix}_${name}_infra2_joint" type="fixed">
       <origin xyz="0 ${d435_cam_depth_to_infra2_offset} 0" rpy="0 0 0" />
-      <parent link="${name}_link" />
-      <child link="${name}_infra2_frame" />
+      <parent link="${prefix}_${name}_link" />
+      <child link="${prefix}_${name}_infra2_frame" />
     </joint>
-    <link name="${name}_infra2_frame"/>
-    <joint name="${name}_infra2_optical_joint" type="fixed">
+    <link name="${prefix}_${name}_infra2_frame"/>
+    <joint name="${prefix}_${name}_infra2_optical_joint" type="fixed">
       <origin xyz="0 0 0" rpy="${-M_PI/2} 0 ${-M_PI/2}" />
-      <parent link="${name}_infra2_frame" />
-      <child link="${name}_infra2_optical_frame" />
+      <parent link="${prefix}_${name}_infra2_frame" />
+      <child link="${prefix}_${name}_infra2_optical_frame" />
     </joint>
-    <link name="${name}_infra2_optical_frame"/>
+    <link name="${prefix}_${name}_infra2_optical_frame"/>
     <!-- camera color joints and links -->
-    <joint name="${name}_color_joint" type="fixed">
+    <joint name="${prefix}_${name}_color_joint" type="fixed">
       <origin xyz="0 ${d435_cam_depth_to_color_offset} 0" rpy="0 0 0" />
-      <parent link="${name}_link" />
-      <child link="${name}_color_frame" />
+      <parent link="${prefix}_${name}_link" />
+      <child link="${prefix}_${name}_color_frame" />
     </joint>
-    <link name="${name}_color_frame"/>
-    <joint name="${name}_color_optical_joint" type="fixed">
+    <link name="${prefix}_${name}_color_frame"/>
+    <joint name="${prefix}_${name}_color_optical_joint" type="fixed">
       <origin xyz="0 0 0" rpy="${-M_PI/2} 0 ${-M_PI/2}" />
-      <parent link="${name}_color_frame" />
-      <child link="${name}_color_optical_frame" />
+      <parent link="${prefix}_${name}_color_frame" />
+      <child link="${prefix}_${name}_color_optical_frame" />
     </joint>
-    <link name="${name}_color_optical_frame"/>
+    <link name="${prefix}_${name}_color_optical_frame"/>
     <!--/xacro:if-->
     <!-- Gazebo part -->
