Commit message: update for macro template

File: summit_xls/summit_xls_franka_sim/urdf/roas.urdf.xacro (robot description, xacro)
@@ -1,70 +1,72 @@
 <?xml version="1.0"?>
 <robot xmlns:xacro="http://ros.org/wiki/xacro" name="roas">
-  <xacro:property name="PI" value="3.1415926535897931"/>
-  <xacro:include filename="$(find summit_xls_franka_sim)/urdf/d435.urdf.xacro"/>
-  <link name="top_structure">
-    <visual>
-      <origin xyz="0 0 0" rpy="0 0 0" />
-      <geometry>
-        <mesh filename="package://summit_xl_description/meshes/structures/top_structure_roas.STL"/>
-      </geometry>
-      <material name="silver">
-        <color rgba="0.75 0.75 0.75 1"/>
-      </material>
-    </visual>
-    <collision>
+  <xacro:macro name="roas" params="prefix">
+    <xacro:property name="PI" value="3.1415926535897931"/>
+    <xacro:include filename="$(find summit_xls_franka_sim)/urdf/d435.urdf.xacro"/>
+    <link name="${prefix}_top_structure">
+      <visual>
+        <origin xyz="0 0 0" rpy="0 0 0" />
+        <geometry>
+          <mesh filename="package://summit_xl_description/meshes/structures/top_structure_roas.STL"/>
+        </geometry>
+        <material name="silver">
+          <color rgba="0.75 0.75 0.75 1"/>
+        </material>
+      </visual>
+      <collision>
+        <origin xyz="0 0 0" rpy="0 0 0"/>
+        <geometry>
+          <mesh filename="package://summit_xl_description/meshes/structures/top_structure_roas.STL"/>
+        </geometry>
+      </collision>
+    </link>
+    <xacro:include filename="$(find summit_xls_franka_sim)/urdf/arm/fr3.urdf.xacro"/>
+    <!-- fr3 -->
+    <joint name="${prefix}_fr3_base_joint" type="fixed">
+      <origin xyz="0.23 0 0.66" rpy="0 0 0"/>
+      <parent link="${prefix}_top_structure"/>
+      <child link="${prefix}_fr3_link0"/>
+    </joint>
+    <link name="${prefix}_ee_link"/>
+    <joint name="${prefix}_ee_joint" type="fixed">
+      <parent link="${prefix}_fr3_link8" />
+      <child link="${prefix}_ee_link" />
       <origin xyz="0 0 0" rpy="0 0 0"/>
-      <geometry>
-        <mesh filename="package://summit_xl_description/meshes/structures/top_structure_roas.STL"/>
-      </geometry>
-    </collision>
-  </link>
-  <xacro:include filename="$(find summit_xls_franka_sim)/urdf/arm/fr3.urdf.xacro"/>
-  <!-- fr3 -->
-  <joint name="fr3_base_joint" type="fixed">
-    <origin xyz="0.23 0 0.66" rpy="0 0 0"/>
-    <parent link="top_structure"/>
-    <child link="fr3_link0"/>
-  </joint>
-  <link name="ee_link"/>
-  <joint name="ee_joint" type="fixed">
-    <parent link="fr3_link8" />
-    <child link="ee_link" />
-    <origin xyz="0 0 0" rpy="0 0 0"/>
-  </joint>
-  <!-- D435 -->
-  <xacro:sensor_d435 parent="camera_bracket" name="camera">
-    <origin xyz="0.0377 0 0.0105" rpy="0 -1.57 3.14"/>
-  </xacro:sensor_d435>
-  <link name="d435_link"/>
-  <joint name="d435_joint" type="fixed">
-    <parent link="camera_link"/>
-    <child link="d435_link"/>
-    <origin xyz="0.0 0.0 0.0" rpy="-${PI/2} 0 -${PI/2}"/>
-  </joint>
-  <link name="camera_bracket">
-    <visual>
-      <origin xyz="0 0 0" rpy="0 0 0" />
-      <geometry>
-        <mesh filename="package://summit_xl_description/meshes/structures/hand_camera.STL"/>
-      </geometry>
-      <material name="silver">
-        <color rgba="0.75 0.75 0.75 1"/>
-      </material>
-    </visual>
-    <collision>
-      <origin xyz="0 0 0" rpy="0 0 0" />
-      <geometry>
-        <mesh filename="package://summit_xl_description/meshes/structures/hand_camera.STL"/>
-      </geometry>
-      <material name="silver">
-        <color rgba="0.75 0.75 0.75 1"/>
-      </material>
-    </collision>
-  </link>
-  <joint name="camera_bracket_joint" type="fixed">
-    <parent link="ee_link" />
-    <child link = "camera_bracket" />
-    <origin xyz="0 0 0.003" rpy="0 0 -0.785" />
-  </joint>
+    </joint>
+    <!-- D435 -->
+    <xacro:sensor_d435 parent="${prefix}_camera_bracket" name="camera">
+      <origin xyz="0.0377 0 0.0105" rpy="0 -1.57 3.14"/>
+    </xacro:sensor_d435>
+    <link name="${prefix}_d435_link"/>
+    <joint name="${prefix}_d435_joint" type="fixed">
+      <parent link="${prefix}_camera_link"/>
+      <child link="${prefix}_d435_link"/>
+      <origin xyz="0.0 0.0 0.0" rpy="-${PI/2} 0 -${PI/2}"/>
+    </joint>
+    <link name="${prefix}_camera_bracket">
+      <visual>
+        <origin xyz="0 0 0" rpy="0 0 0" />
+        <geometry>
+          <mesh filename="package://summit_xl_description/meshes/structures/hand_camera.STL"/>
+        </geometry>
+        <material name="silver">
+          <color rgba="0.75 0.75 0.75 1"/>
+        </material>
+      </visual>
+      <collision>
+        <origin xyz="0 0 0" rpy="0 0 0" />
+        <geometry>
+          <mesh filename="package://summit_xl_description/meshes/structures/hand_camera.STL"/>
+        </geometry>
+        <material name="silver">
+          <color rgba="0.75 0.75 0.75 1"/>
+        </material>
+      </collision>
+    </link>
+    <joint name="${prefix}_camera_bracket_joint" type="fixed">
+      <parent link="${prefix}_ee_link" />
+      <child link = "${prefix}_camera_bracket" />
+      <origin xyz="0 0 0.003" rpy="0 0 -0.785" />
+    </joint>
+  </xacro:macro>
 </robot>

File: summit_xls/summit_xls_franka_sim/urdf/summit_xls_franka_std.urdf.xacro (robot description, xacro)
@@ -12,5 +12,5 @@
 	<xacro:include filename="$(find summit_xl_description)/urdf/structures/structure_hokuyo.urdf.xacro" />
 	<!-- Import all available sensors -->
-	<xacro:include filename="$(find robotnik_sensors)/urdf/all_sensors.urdf.xacro" />
+	<!-- <xacro:include filename="$(find robotnik_sensors)/urdf/all_sensors.urdf.xacro" /> -->
 	<xacro:property name="PI" value="3.1415926535897931"/>
 	<!-- Wheel parameters -->

File: summit_xls_franka_base.urdf.xacro (robot description, xacro)
@@ -8,5 +8,5 @@
 	<!-- BASE FOOTPRINT -->
 	  <xacro:if value="${publish_bf}">
-		<link name="${prefix}_base_footprint">
+		<link name="${prefix}base_footprint">
 		  <visual>
 			  <origin xyz="0 0 0" rpy="0 0 0" />
@@ -16,12 +16,12 @@
 		  </visual>
 		</link>
-		<joint name="${prefix}_base_footprint_joint" type="fixed">
+		<joint name="${prefix}base_footprint_joint" type="fixed">
 		  <origin xyz="0 0 ${wheel_radius}" rpy="0 0 0" /> <!-- ${wheel_radius} property must be defined inside wheel description -->
-		  <parent link="${prefix}_base_footprint"/>
-		  <child link="${prefix}_base_link" />
+		  <parent link="${prefix}base_footprint"/>
+		  <child link="${prefix}base_link" />
 		</joint>
 	  </xacro:if>
   <!-- BASE_LINK -->
-  <link name="${prefix}_base_link">
+  <link name="${prefix}base_link">
     <inertial>
       <mass value="125.0" />  <!-- origin : 125.0 -->
@@ -52,9 +52,9 @@
     </collision>
   </link>
-  <gazebo reference="${prefix}_base_link">
+  <gazebo reference="${prefix}base_link">
     <material>Gazebo/Black</material>
   </gazebo>
   <!-- CHAPAS INOX TAPAS -->
-  <link name="${prefix}_base_chapa">
+  <link name="${prefix}base_chapa">
   <visual>
     <origin xyz="0 0 0" rpy="0 0 0" />
@@ -67,11 +67,11 @@
     </visual>
   </link>
-  <joint name="${prefix}_base_tapa_joint" type="fixed">
+  <joint name="${prefix}base_tapa_joint" type="fixed">
     <origin xyz="0.0 0 0.38062" rpy="0 0 0" />
-    <parent link="${prefix}_base_link"/>
-    <child link="${prefix}_base_chapa" />
+    <parent link="${prefix}base_link"/>
+    <child link="${prefix}base_chapa" />
   </joint>
   <!-- LOGO ROBOTNIK IZQUIERDO -->
-  <link name="${prefix}_base_logo_left">
+  <link name="${prefix}base_logo_left">
   <visual>
     <origin xyz="0 0 0" rpy="0 0 0" />
@@ -84,11 +84,11 @@
     </visual>
   </link>
-  <joint name="${prefix}_base_logo_left_joint" type="fixed">
+  <joint name="${prefix}base_logo_left_joint" type="fixed">
     <origin xyz="0.0 0.28931 0.29062" rpy="0 0 0" />
-    <parent link="${prefix}_base_link"/>
-    <child link="${prefix}_base_logo_left" />
+    <parent link="${prefix}base_link"/>
+    <child link="${prefix}base_logo_left" />
   </joint>
   <!-- LOGO ROBOTNIK DERECHO -->
-  <link name="${prefix}_base_logo_right">
+  <link name="${prefix}base_logo_right">
   <visual>
     <origin xyz="0 0 0" rpy="0 0 0" />
@@ -101,11 +101,11 @@
     </visual>
   </link>
-  <joint name="${prefix}_base_logo_right_joint" type="fixed">
+  <joint name="${prefix}base_logo_right_joint" type="fixed">
     <origin xyz="0.0 -0.28931 0.29062" rpy="0 0 ${PI}" />
-    <parent link="${prefix}_base_link"/>
-    <child link="${prefix}_base_logo_right" />
+    <parent link="${prefix}base_link"/>
+    <child link="${prefix}base_logo_right" />
   </joint>
   <!-- LOGO ROBOTNIK FRONTAL -->
-  <link name="${prefix}_base_logo_front">
+  <link name="${prefix}base_logo_front">
   <visual>
     <origin xyz="0 0 0" rpy="0 0 0" />
@@ -118,11 +118,11 @@
     </visual>
   </link>
-  <joint name="${prefix}_base_logo_front_joint" type="fixed">
+  <joint name="${prefix}base_logo_front_joint" type="fixed">
     <origin xyz="0.345 0.0 0.0" rpy="0 0 ${-PI/2}" />
-    <parent link="${prefix}_base_link"/>
-    <child link="${prefix}_base_logo_front" />
+    <parent link="${prefix}base_link"/>
+    <child link="${prefix}base_logo_front" />
   </joint>
   <!-- LOGO ROBOTNIK TRASERO -->
-  <link name="${prefix}_base_logo_rear">
+  <link name="${prefix}base_logo_rear">
   <visual>
     <origin xyz="0 0 0" rpy="0 0 0" />
@@ -135,23 +135,22 @@
     </visual>
   </link>
-  <joint name="${prefix}_base_logo_rear_joint" type="fixed">
+  <joint name="${prefix}base_logo_rear_joint" type="fixed">
     <origin xyz="-0.345 0.0 0.0" rpy="0 0 ${PI/2}" />
-    <parent link="${prefix}_base_link"/>
-    <child link="${prefix}_base_logo_rear" />
+    <parent link="${prefix}base_link"/>
+    <child link="${prefix}base_logo_rear" />
   </joint>
    <!-- DOCKING CONTACT -->
-    <link name="${prefix}_base_docking_contact">
+    <link name="${prefix}base_docking_contact">
     </link>
-    <joint name="${prefix}_base_docking_joint" type="fixed">
+    <joint name="${prefix}base_docking_joint" type="fixed">
       <origin xyz="0.35 0 0.09" rpy="0 0 0" />
-      <parent link="${prefix}_base_link"/>
-      <child link="${prefix}_base_docking_contact" />
+      <parent link="${prefix}base_link"/>
+      <child link="${prefix}base_docking_contact" />
     </joint>
   <xacro:include filename="$(find summit_xl_description)/urdf/structures/roas.urdf.xacro"/>
-  <xacro:roas prefix="${prefix}"/>
-  <joint name="${prefix}_top_structure_joint" type="fixed">
+  <joint name="top_structure_joint" type="fixed">
     <origin xyz="0 0 0" rpy="0 0 0" />
-    <parent link="${prefix}_base_footprint"/>
-    <child link="${prefix}_top_structure" />
+    <parent link="${prefix}base_footprint"/>
+    <child link="top_structure" />
   </joint>
   </xacro:macro>
